Commit message: catkin_ws from tractor laptop 2022-11-23

File: src/lawn_tractor_sim/urdf/lawn_tractor.urdf.xacro (robot description, xacro)
@@ -8,5 +8,5 @@
       <origin xyz='0.55 0 0' rpy='0 0 ${pi}' />
       <geometry>
-        <mesh filename="package://lawn_tractor_sim/meshes/lawn_tractor.dae" scale='1 1 1'/>
+        <mesh filename="package://home/tractor/catkin_ws/src/lawn_tractor_sim/meshes/lawn_tractor.dae" scale='1 1 1'/>
       </geometry>
     </visual>

Commit message: catkin_ws from tractor laptop 2022-11-23 5pm

File: src/lawn_tractor_sim/urdf/lawn_tractor.urdf.xacro (robot description, xacro)
@@ -8,5 +8,5 @@
       <origin xyz='0.55 0 0' rpy='0 0 ${pi}' />
       <geometry>
-        <mesh filename="package://home/tractor/catkin_ws/src/lawn_tractor_sim/meshes/lawn_tractor.dae" scale='1 1 1'/>
+        <mesh filename="file:/home/tractor/catkin_ws/src/lawn_tractor_sim/meshes/lawn_tractor.dae" scale='1 1 1'/>
       </geometry>
     </visual>
