Commit message: catkin_ws from tractor laptop 2023-01-07

File: src/picar/src/ackermann_vehicle_description/urdf/ack_new_macros.xacro (robot description, xacro)
@@ -56,5 +56,7 @@
         <parent link="base_footprint"/>
         <child link="base_link"/>
-        <origin xyz="0.0 0 0.1525"/>
+       <!--  <origin xyz="0.0 0 0.1525"/> -->
+       <!-- <origin xyz="0.0 0 ${tire_rear_dia}"/>  wheels are still off the ground -->
+        <origin xyz="0.0 0 ${tire_rear_dia / 2}"/>
     </joint>
     <link name="base_link">

File: src/picar/src/ackermann_vehicle_description/urdf/robot_core.xacro (robot description, xacro)
@@ -21,4 +21,5 @@
         <parent link="base_link"/>
         <child link="chassis"/>
+        <!-- <origin xyz="-0.1 0 0"/> the vehicle was suspended in air-->
         <origin xyz="-0.1 0 0"/>
     </joint>
